File: Eagle/Arduinoboy.brd (EAGLE design)
At the start: 68.6 x 53.3 mm, 20 parts

Commit message: Revert "Merge branch 'master' into ps2"
This reverts commit 4c279bdc1415769d58dcdb31e5e95ad5c8d64dd7, reversing
changes made to 2334a322f219572b62a75aed99c683bbc509b818.
Parts:
- moved U$2 2.07 mm to (66.0, 17.8)
Routing:
- net N$9: track 88.4 -> 65.8 mm
- net N$16: track 44.1 -> 30.1 mm, vias 0 -> 2
- net N$19: track 84.8 -> 71.5 mm
- net N$11: track 38.0 -> 25.4 mm
- net VCC: track 95.6 -> 85.4 mm
- net N$4: track 128.1 -> 122.1 mm
- net N$14: track 47.4 -> 42.9 mm
- net N$13: track 26.8 -> 30.3 mm
- net N$7: track 43.2 -> 41.2 mm
- net GND: track 133.6 -> 131.9 mm
- net N$21: track 55.5 -> 56.6 mm
- net N$8: track 24.1 -> 25.1 mm
- net N$20: track 57.6 -> 58.2 mm
- net N$5: vias 0 -> 1
Other:
- board text added: "1.1.0"
- board text removed: "1.1.1"

Commit message: Update to master
Parts:
- moved U$2 2.07 mm to (66.1, 15.7)
- renumbered KEYBRD to KB, MGBOY to MGB, NLOOP to NL
Connections:
- removed net N$20: U$1.SI, U$3.A2, X1.1
- new net N$22: U$1.SI, U$3.A2
- net N$21: now also X1.1
Routing:
- net N$20: track 58.2 -> 0.00 mm
- net N$22: track 0.00 -> 58.1 mm
- net N$9: track 65.8 -> 44.0 mm, vias 0 -> 2
- net N$8: track 25.1 -> 43.7 mm
- net VCC: track 85.4 -> 70.4 mm, vias 0 -> 1
- net N$16: track 30.1 -> 44.1 mm, vias 2 -> 0
- net N$11: track 25.4 -> 38.2 mm
- net GND: track 131.9 -> 141.7 mm, vias 1 -> 12
- net N$19: track 71.5 -> 78.9 mm
- net N$4: track 122.1 -> 128.5 mm
- net N$14: track 42.9 -> 47.4 mm
- net N$13: track 30.3 -> 26.8 mm
- net N$18: track 45.8 -> 48.3 mm
- net N$7: track 41.2 -> 43.2 mm
- net N$17: track 52.1 -> 52.8 mm
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Other:
- board text added: "1.1.3"
- board text removed: "1.1.0"
